Commit message: Enable hw interface to be passed as argument

File: robotiq_2f_140_gripper_visualization/urdf/robotiq_arg2f_140_model_macro.xacro (robot description, xacro)
@@ -204,5 +204,5 @@
     <xacro:finger_joints prefix="${prefix}" fingerprefix="right" reflect="-1.0"/>
   </xacro:macro>
-  <xacro:macro name="robotiq_arg2f_140" params="prefix">
+  <xacro:macro name="robotiq_arg2f_140" params="prefix robotiq_transmission_hw_interface">
     <xacro:robotiq_arg2f_base_link prefix="${prefix}"/>
     <xacro:finger_links prefix="${prefix}" fingerprefix="left" stroke="140"/>
@@ -210,5 +210,5 @@
     <xacro:finger_joint prefix="${prefix}"/>
     <xacro:right_outer_knuckle_joint prefix="${prefix}"/>
-    <xacro:robotiq_arg2f_transmission prefix="${prefix}"/>
+    <xacro:robotiq_arg2f_transmission prefix="${prefix}" hw_interface="${robotiq_transmission_hw_interface}" />
     <xacro:robotiq_arg2f_gazebo prefix="${prefix}"/>
   </xacro:macro>
