Commit message: Update gazebo mimic plugin call

File: robotiq_2f_140_gripper_visualization/urdf/robotiq_arg2f.gazebo.xacro (robot description, xacro)
@@ -5,5 +5,5 @@
     <!--https://github.com/ros-industrial/robotiq/issues/150-->
         <gazebo>
-            <plugin filename="libroboticsgroup_gazebo_mimic_joint_plugin.so" name="${prefix}mimic_robotiq_140_1">
+            <plugin filename="libroboticsgroup_upatras_gazebo_mimic_joint_plugin.so" name="${prefix}mimic_robotiq_140_1">
                 <joint>${prefix}finger_joint</joint>
                 <mimicJoint>${prefix}right_outer_knuckle_joint</mimicJoint>
@@ -11,5 +11,5 @@
                 <offset>0.0</offset>
             </plugin>
-            <plugin filename="libroboticsgroup_gazebo_mimic_joint_plugin.so" name="${prefix}mimic_robotiq_140_2">
+            <plugin filename="libroboticsgroup_upatras_gazebo_mimic_joint_plugin.so" name="${prefix}mimic_robotiq_140_2">
                 <joint>${prefix}finger_joint</joint>
                 <mimicJoint>${prefix}left_inner_knuckle_joint</mimicJoint>
@@ -17,5 +17,5 @@
                 <offset>0.0</offset>
             </plugin>
-            <plugin filename="libroboticsgroup_gazebo_mimic_joint_plugin.so" name="${prefix}mimic_robotiq_140_3">
+            <plugin filename="libroboticsgroup_upatras_gazebo_mimic_joint_plugin.so" name="${prefix}mimic_robotiq_140_3">
                 <joint>${prefix}finger_joint</joint>
                 <mimicJoint>${prefix}right_inner_knuckle_joint</mimicJoint>
@@ -23,5 +23,5 @@
                 <offset>0.0</offset>
             </plugin>
-            <plugin filename="libroboticsgroup_gazebo_mimic_joint_plugin.so" name="${prefix}mimic_robotiq_140_4">
+            <plugin filename="libroboticsgroup_upatras_gazebo_mimic_joint_plugin.so" name="${prefix}mimic_robotiq_140_4">
                 <joint>${prefix}finger_joint</joint>
                 <mimicJoint>${prefix}left_inner_finger_joint</mimicJoint>
@@ -29,5 +29,5 @@
                 <offset>0.0</offset>
             </plugin>
-            <plugin filename="libroboticsgroup_gazebo_mimic_joint_plugin.so" name="${prefix}mimic_robotiq_140_5">
+            <plugin filename="libroboticsgroup_upatras_gazebo_mimic_joint_plugin.so" name="${prefix}mimic_robotiq_140_5">
                 <joint>${prefix}finger_joint</joint>
                 <mimicJoint>${prefix}right_inner_finger_joint</mimicJoint>

File: robotiq_2f_140_gripper_visualization/urdf/robotiq_arg2f_140_model_macro.xacro (robot description, xacro)
@@ -204,5 +204,6 @@
     <xacro:finger_joints prefix="${prefix}" fingerprefix="right" reflect="-1.0"/>
   </xacro:macro>
-  <xacro:macro name="robotiq_arg2f_140" params="prefix robotiq_transmission_hw_interface">
+  <xacro:macro name="robotiq_arg2f_140" params="prefix
+    robotiq_transmission_hw_interface:=EffortJointInterface">
     <xacro:robotiq_arg2f_base_link prefix="${prefix}"/>
     <xacro:finger_links prefix="${prefix}" fingerprefix="left" stroke="140"/>

Commit message: Render gripper color in Gazebo

File: robotiq_2f_140_gripper_visualization/urdf/robotiq_arg2f.gazebo.xacro (robot description, xacro)
@@ -37,3 +37,15 @@
         </gazebo>
     </xacro:macro>
+    <xacro:macro name="robotiq_gazebo_ref" params="append_prefix:=true prefix fingerprefix link color">
+        <xacro:if value="${append_prefix}">
+            <gazebo reference="${prefix}${fingerprefix}_${link}">
+                <material>${color}</material>
+            </gazebo>
+        </xacro:if>
+        <xacro:unless value="${append_prefix}">
+            <gazebo reference="${link}">
+                <material>${color}</material>
+            </gazebo>
+        </xacro:unless>
+    </xacro:macro>
 </robot>
