Commit message: restructured robotiq_arg2f_gripper_visualization

File: robotiq_2f_140_gripper_visualization/urdf/inc/robotiq_arg2f_140_transmissions.xacro (robot description, xacro)
@@ -1,5 +1,5 @@
 <?xml version="1.0"?>
 <robot xmlns:xacro="http://wiki.ros.org/xacro">
-  <xacro:macro name="robotiq_arg2f_transmission" params="prefix hw_interface">
+  <xacro:macro name="robotiq_arg2f_140_transmission" params="prefix hw_interface">
     <transmission name="${prefix}finger_joint_trans">
       <type>transmission_interface/SimpleTransmission</type>
